File: Hardware/Module++/Module++.kicad_pcb (KiCad board)
At the start: 2 copper layers, 90 x 30 mm, 17 parts, among them J1 CONN_01X01, J2 CONN_02X03, J3 CONN_01X04, J4 CONN_02X03, J5 CONN_01X04, J6 CONN_01X01, U1 74LS353

Commit message: Hardware: Fix missing VCC connection
Signed-off-by: Paul Kocialkowski <contact@paulk.fr>
Routing:
- net VCC: track 115.5 -> 140.4 mm
Changed lines of the file:
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@@
     (links 40)
     (no_connects 1)
-    (area 127.164999 53.504999 217.315001 83.655001)
+    (area 126.525 52.575 217.315001 83.820001)
     (thickness 1.6)
     (drawings 6)
-    (tracks 131)
+    (tracks 139)
     (zones 0)
     (modules 17)
@@
   (segment (start 129 59.8) (end 129 58.8) (width 0.25) (layer F.Cu) (net 1))
   (segment (start 129 58.8) (end 129 57.9) (width 0.25) (layer F.Cu) (net 1))
+  (segment (start 145.8 54.2) (end 132.075 54.2) (width 0.25) (layer F.Cu) (net 2))
+  (segment (start 132.075 54.2) (end 131.225 55.05) (width 0.25) (layer F.Cu) (net 2))
+  (segment (start 131.225 55.05) (end 131.225 56.05) (width 0.25) (layer F.Cu) (net 2))
+  (segment (start 146.6 55) (end 145.8 54.2) (width 0.25) (layer F.Cu) (net 2))
+  (segment (start 146.6 58.97) (end 146.6 55.6) (width 0.25) (layer F.Cu) (net 2))
+  (segment (start 146.6 55.6) (end 146.6 55) (width 0.25) (layer F.Cu) (net 2))
+  (segment (start 143.51 60.96) (end 144.61 60.96) (width 0.25) (layer F.Cu) (net 2))
+  (segment (start 144.61 60.96) (end 146.6 58.97) (width 0.25) (layer F.Cu) (net 2))
   (segment (start 197.16 66.04) (end 139.53 66.04) (width 0.25) (layer F.Cu) (net 2))
   (segment (start 139.53 66.04) (end 138.43 67.14) (width 0.25) (layer F.Cu) (net 2))
@@
     (connect_pads (clearance 0.508))
     (min_thickness 0.254)
-    (fill yes (arc_segments 16) (thermal_gap 0.508) (thermal_bridge_width 0.508))
+    (fill (arc_segments 16) (thermal_gap 0.508) (thermal_bridge_width 0.508))
     (polygon
       (pts
@@
     (connect_pads (clearance 0.508))
     (min_thickness 0.254)
-    (fill yes (arc_segments 16) (thermal_gap 0.508) (thermal_bridge_width 0.508))
+    (fill (arc_segments 16) (thermal_gap 0.508) (thermal_bridge_width 0.508))
     (polygon
       (pts
